File: ergl.sch (KiCad schematic (older format))
At the start: 60 parts, among them J1 CONN_02, J2 CONN_01, J3 AUDIO_JACK_TRRSSMD_RA, J4 CONN_03, J5 0548190519, J6 CONN_04, J7 CONN_02, J8 CONN_01, K1 KEYSW, K10 KEYSW, K11 KEYSW, K12 KEYSW, K13 KEYSW, K14 KEYSW, K15 KEYSW, K16 KEYSW, K17 KEYSW, K18 KEYSW, K19 KEYSW, K2 KEYSW, K20 KEYSW, K21 KEYSW, K22 KEYSW, K23 KEYSW, K24 KEYSW, K25 KEYSW, K3 KEYSW, K4 KEYSW, K5 KEYSW, K6 KEYSW, K7 KEYSW, K8 KEYSW, K9 KEYSW, SW1 RESET BTN, U1 ProMicro

Commit message: pushing up prototype PCB
Parts:
- removed J5: 0548190519, digikey-footprints:USB_Mini_B_Female_548190519, symbol dk_USB-DVI-HDMI-Connectors:0548190519
- removed J6: CONN_04, Connectors:1X04, symbol SparkFun-Connectors:CONN_04
- D1, D10, D11, D12, D13, D14, D15, D16, D17, D18, D19, D2, D20, D21, D22, D23, D24, D25, D3, D4, D5, D6, D7, D8, D9: footprint keyboard_parts:D_axial -> keyboard_parts:D_SOD123_axial
- SW1: footprint digikey-footprints:Switch_Tactile_SMD_4.5x4.5mm_TL3315NF160Q -> Button_Switch_SMD:SW_Push_1P1T_NO_CK_KSC6xxJ
Connections:
- net labels added: pdt1, rst, rx, tx, xd1
- wire segments 88 -> 71
- no-connect marks 3 -> 2
Other:
- moved on the sheet: J2, J8
